File: traced-pcbs/v2/pcbLeft.kicad_pcb (KiCad board)
At the start: 2 copper layers, 146.5 x 126.3 mm, 91 parts

Commit message: General housekeeping
Parts:
- removed ?: , RP2040-Zero
- added JST1: , ceoloide:battery_connector_jst_ph_2, F.Cu at (55.0, 192.6)
- added MCU1: , ProMicro, F.Cu at (41.5, 99.5)
- added PWR1: , ceoloide:power_switch_smd_side, B.Cu at (25.5, 142.0)
- added PinHeader 6Pin1: , PinHeader_1x06_P2.54mm_Vertical, F.Cu at (148.0, 152.4)
- added RST1: , ceoloide:reset_switch_smd_side, B.Cu at (25.5, 123.0)
- added USB-C 16 Pin Receptacle1: , USB_C_Receptacle_XKB_U262-16XN-4BVC11, F.Cu at (135.0, 93.3)
- moved LOGO1 72.2 mm to (33.5, 192.5)
- moved MH6 13.4 mm to (103.0, 175.9)
- moved MH3 7.60 mm to (61.0, 93.4)
- moved MH4 5.50 mm to (27.0, 112.5)
Connections:
- net GP10 renamed P3
- net GP11 renamed P4
- net GP12 renamed P5
- net GP13 renamed P6
- net GP14 renamed P14
- net GP15 renamed P15
- net GP26 renamed P18
- net GP27 renamed P19
- net GP28 renamed P20
- net GP29 renamed P21
- net GP9 renamed P2
- LED1 pad 1: P5V -> RAW
- LED1 pad 4: GP2 -> P7
- LED10 pad 1: P5V -> RAW
- LED11 pad 1: P5V -> RAW
- LED12 pad 1: P5V -> RAW
- LED13 pad 1: P5V -> RAW
- LED14 pad 1: P5V -> RAW
- LED15 pad 1: P5V -> RAW
- LED16 pad 1: P5V -> RAW
- LED17 pad 1: P5V -> RAW
- LED18 pad 1: P5V -> RAW
- LED19 pad 1: P5V -> RAW
- LED2 pad 1: P5V -> RAW
- LED20 pad 1: P5V -> RAW
- LED21 pad 1: P5V -> RAW
- LED22 pad 1: P5V -> RAW
- LED23 pad 1: P5V -> RAW
- LED24 pad 1: P5V -> RAW
- LED25 pad 1: P5V -> RAW
- LED26 pad 1: P5V -> RAW
- LED27 pad 1: P5V -> RAW
- LED27 pad 2: GP3 -> undefined
- LED3 pad 1: P5V -> RAW
- LED4 pad 1: P5V -> RAW
- LED5 pad 1: P5V -> RAW
- LED6 pad 1: P5V -> RAW
- LED7 pad 1: P5V -> RAW
- LED8 pad 1: P5V -> RAW
- LED9 pad 1: P5V -> RAW
- USB 4p Breakout1 pad 1: P3V3 -> RAW
- USB 4p Breakout1 pad 2: GP0 -> P1
- USB 4p Breakout1 pad 3: GP1 -> P0
Routing:
- net RAW: track 0.00 -> 1159.0 mm, vias 0 -> 31
- net P5V: track 883.6 -> 0.00 mm, vias 32 -> 0
- net GP3: track 236.8 -> 0.00 mm, vias 2 -> 0
- net P16: track 0.00 -> 176.6 mm
- net P10: track 0.00 -> 170.3 mm
- net P8: track 0.00 -> 161.2 mm, vias 0 -> 1
- net P9: track 0.00 -> 159.9 mm
- net P3V3: track 135.2 -> 0.00 mm, vias 1 -> 0
- net P1: track 0.00 -> 125.2 mm
- net P0: track 0.00 -> 124.6 mm
- net GP0: track 119.6 -> 0.00 mm, vias 1 -> 0
- net GP1: track 117.4 -> 0.00 mm, vias 1 -> 0
- net GND: track 902.3 -> 998.3 mm, vias 32 -> 35
- net P2: track 275.5 -> 184.8 mm, vias 7 -> 6
- net BAT_P: track 0.00 -> 85.3 mm
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Other:
- outline, holes or cut-outs redrawn
- board text added: "Battery goes here ↓ Max Dimentions: 34mm x 18.5mm x 8mm"
