File: traced-pcbs/v2/pcbRight.kicad_pcb (KiCad board)
At the start: 2 copper layers, 146.5 x 126.3 mm, 91 parts

Commit message: General housekeeping
Parts:
- removed ?: , RP2040-Zero
- added JST1: , ceoloide:battery_connector_jst_ph_2, F.Cu at (333.0, 192.6)
- added MCU1: , ProMicro, F.Cu at (346.5, 99.5)
- added PWR1: , ceoloide:power_switch_smd_side, B.Cu at (362.5, 142.0)
- added PinHeader 6Pin1: , PinHeader_1x06_P2.54mm_Vertical, F.Cu at (240.0, 165.1)
- added RST1: , ceoloide:reset_switch_smd_side, B.Cu at (362.5, 123.0)
- added USB-C 16 Pin Receptacle1: , USB_C_Receptacle_XKB_U262-16XN-4BVC11, F.Cu at (253.0, 93.3)
- moved LOGO1 72.2 mm to (354.5, 192.5)
- moved LED13 22.6 mm to (272.0, 187.4), turned to 180 degrees
- moved LED26 22.6 mm to (249.6, 190.3), turned to -165 degrees
- moved MH6 13.4 mm to (285.0, 175.9)
- moved MH3 7.60 mm to (327.0, 93.4)
- moved MH4 5.50 mm to (361.0, 112.5)
Connections:
- net GP10 renamed P3
- net GP11 renamed P4
- net GP12 renamed P5
- net GP13 renamed P6
- net GP14 renamed P14
- net GP15 renamed P15
- net GP26 renamed P18
- net GP27 renamed P19
- net GP28 renamed P20
- net GP29 renamed P21
- net GP9 renamed P2
- LED1 pad 1: P5V -> RAW
- LED1 pad 4: GP2 -> P7
- LED10 pad 1: P5V -> RAW
- LED11 pad 1: P5V -> RAW
- LED12 pad 1: P5V -> RAW
- LED13 pad 1: P5V -> RAW
- LED13 pad 2: LED_IN -> LED_OUT
- LED13 pad 4: LED_OUT -> LED_IN
- LED14 pad 1: P5V -> RAW
- LED15 pad 1: P5V -> RAW
- LED16 pad 1: P5V -> RAW
- LED17 pad 1: P5V -> RAW
- LED18 pad 1: P5V -> RAW
- LED19 pad 1: P5V -> RAW
- LED2 pad 1: P5V -> RAW
- LED20 pad 1: P5V -> RAW
- LED21 pad 1: P5V -> RAW
- LED22 pad 1: P5V -> RAW
- LED23 pad 1: P5V -> RAW
- LED24 pad 1: P5V -> RAW
- LED25 pad 1: P5V -> RAW
- LED26 pad 1: P5V -> RAW
- LED26 pad 2: LED_OUT -> LED_IN
- LED26 pad 4: LED_IN -> LED_OUT
- LED27 pad 1: P5V -> RAW
- LED27 pad 2: GP3 -> undefined
- LED3 pad 1: P5V -> RAW
- LED4 pad 1: P5V -> RAW
- LED5 pad 1: P5V -> RAW
- LED6 pad 1: P5V -> RAW
- LED7 pad 1: P5V -> RAW
- LED8 pad 1: P5V -> RAW
- LED9 pad 1: P5V -> RAW
- USB 4p Breakout1 pad 1: P3V3 -> RAW
- USB 4p Breakout1 pad 2: GP0 -> P1
- USB 4p Breakout1 pad 3: GP1 -> P0
Routing:
- net RAW: track 0.00 -> 1040.7 mm, vias 0 -> 33
- net P5V: track 905.1 -> 0.00 mm, vias 33 -> 0
- net GP3: track 243.9 -> 0.00 mm, vias 2 -> 0
- net P8: track 0.00 -> 164.6 mm
- net P9: track 0.00 -> 159.8 mm
- net P16: track 0.00 -> 152.4 mm
- net P10: track 0.00 -> 149.8 mm
- net GP0: track 140.9 -> 0.00 mm, vias 2 -> 0
- net GP1: track 139.7 -> 0.00 mm, vias 2 -> 0
- net P1: track 0.00 -> 128.5 mm
- net P3V3: track 121.7 -> 0.00 mm
- net P0: track 0.00 -> 121.1 mm
- net P2: track 258.6 -> 162.4 mm
- net GND: track 995.7 -> 1082.1 mm, vias 33 -> 35
- net BAT_P: track 0.00 -> 73.1 mm
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Other:
- outline, holes or cut-outs redrawn
- board text added: "Battery goes here ↓ Max Dimentions: 34mm x 18.5mm x 8mm"
